File: strip.kicad_pcb (KiCad board)
At the start: 4 copper layers, 66 x 18 mm, 44 parts, among them J102 WAGO-2065, J103 WAGO-2065, J104 WAGO-2065, J105 CORTEX-DEBUG, J106 JAE DX07S016JA1R1500, SW101 SW_Push, SW102 SW_Push, U101 74AHC1G125, U102 ATSAMD51G, U103 AP2112K-3.3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

Commit message: Update to KiCad 7.0
Parts:
- removed C111: 100n, Capacitor_SMD:C_0603_1608Metric
- removed J102, J103, J104: WAGO-2065, V2_Connector_Wago:WAGO2065-100
- removed U101: 74AHC1G125, Package_TO_SOT_SMD:SOT-23-5
- added J301: WAGO-2065, V2_Connector_WAGO:2065-100, F.Cu at (177.2, 110.0)
- added J302: WAGO-2065, V2_Connector_WAGO:2065-100, F.Cu at (177.2, 103.0)
- added J303: WAGO-2065, V2_Connector_WAGO:2065-100, F.Cu at (177.2, 106.5)
- added U301: 74AHC1G125, Package_TO_SOT_SMD:SOT-23-5, F.Cu at (165.0, 101.0)
- C104, C105, C106, C107, C108, C112: value 100n -> 0u1
- J106: value JAE DX07S016JA1R1500 -> JAE_DX07S016JA3; footprint V2_Connector_USB:JAE_DX07S016JA1R1500 -> V2_Connector_USB:JAE_DX07S016JA3
- SPACER101, SPACER102: value 977?2434030 -> 3mm
- Y101: value 32.768kHz -> 32k768
- moved C110 4.01 mm to (134.5, 111.2)
- moved C109 3.69 mm to (134.5, 109.2), turned to 180 degrees
- moved U103 3.51 mm to (138.0, 110.2), turned to 90 degrees
- moved ICON103 0.10 mm to (172.2, 103.0)
Connections:
- net +3.3V renamed +3V3
- U102 pad 25: /LED-data -> /LED-Data
Routing:
- net /LED-Data: track 0.00 -> 20.9 mm
- net /LED-data: track 20.9 -> 0.00 mm
- net /WS2812-data: track 12.4 -> 0.00 mm
- net /LED Strip/WS2812-data: track 0.00 -> 12.4 mm
- net GND: track 40.0 -> 33.1 mm, vias 40 -> 39
- net +3V3: track 17.3 -> 15.7 mm, vias 10 -> 8
- net +5V: track 18.7 -> 18.5 mm, vias 14 -> 13
