File: strip.kicad_sch (KiCad schematic)
At the start: 44 parts, among them J102 WAGO-2065, J103 WAGO-2065, J104 WAGO-2065, J105 CORTEX-DEBUG, J106 JAE DX07S016JA1R1500, SW101 SW_Push, SW102 SW_Push, U101 74AHC1G125, U102 ATSAMD51G, U103 AP2112K-3.3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

Commit message: Update to KiCad 7.0
Parts:
- removed C111: 100n, Capacitor_SMD:C_0603_1608Metric, symbol Device:C_Small
- removed J102, J103, J104: WAGO-2065, V2_Connector_Wago:WAGO2065-100, symbol V2_Connector:WAGO-2065
- removed U101: 74AHC1G125, Package_TO_SOT_SMD:SOT-23-5, symbol V2_74xGxx:74AHC1G125
- C104, C105, C106, C107, C108, C112: value 100n -> 0u1
- J106: value JAE DX07S016JA1R1500 -> JAE_DX07S016JA3; footprint V2_Connector_USB:JAE_DX07S016JA1R1500 -> V2_Connector_USB:JAE_DX07S016JA3; symbol V2_Connector_USB:JAE_DX07S016JA1R1500 -> V2_Connector_USB:JAE_DX07S016JA3
- SPACER101, SPACER102: value 977?2434030 -> 3mm; symbol V2_Spacer_Wurth:977?2434030 -> V2_Spacer_Wurth:9774030243
- Y101: value 32.768kHz -> 32k768
Connections:
- net +3.3V renamed +3V3
- net LED-data renamed LED-Data
Other:
- added sheet LED Strip (LEDStrip.kicad_sch)
- moved on the sheet: C109, C110, C112, D101, ESD101, J106, R102, R103, R104, R105, U103

Commit message: Refresh
Parts:
- FID101, FID102, FID103: now left out of the parts list
Other:
- moved on the sheet: ICON102
Changed lines of the file:
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@@
   (title_block
     (title "V2 strip")
-    (date "2023-01-12")
+    (date "2023-09-12")
     (rev "3")
     (company "Versio Duo")
@@
       (effects (font (size 1.27 1.27)) hide)
     )
+    (property "Sim.Enable" "0" (at 227.33 152.4 0)
+      (effects (font (size 1.27 1.27)) hide)
+    )
     (instances
       (project "strip"
@@
       (effects (font (size 1.27 1.27)) hide)
     )
+    (property "Sim.Enable" "0" (at 201.93 175.26 0)
+      (effects (font (size 1.27 1.27)) hide)
+    )
     (instances
       (project "strip"
@@
       (effects (font (size 1.27 1.27)) hide)
     )
+    (property "Sim.Enable" "0" (at 201.93 156.21 0)
+      (effects (font (size 1.27 1.27)) hide)
+    )
     (instances
       (project "strip"
@@
       (effects (font (size 1.27 1.27)) hide)
     )
+    (property "Sim.Enable" "0" (at 127 101.6 0)
+      (effects (font (size 1.27 1.27)) hide)
+    )
     (pin "1")
     (pin "10")
@@
       (effects (font (size 1.27 1.27)) hide)
     )
+    (property "Sim.Enable" "0" (at 252.73 152.4 0)
+      (effects (font (size 1.27 1.27)) hide)
+    )
     (pin "1")
     (instances
@@
       (effects (font (size 1.27 1.27)) hide)
     )
+    (property "Sim.Enable" "0" (at 172.72 186.69 0)
+      (effects (font (size 1.27 1.27)) hide)
+    )
     (instances
       (project "strip"
@@
     )
     (property "Datasheet" "" (at 252.73 165.1 0)
+      (effects (font (size 1.27 1.27)) hide)
+    )
+    (property "Sim.Enable" "0" (at 252.73 165.1 0)
       (effects (font (size 1.27 1.27)) hide)
     )
@@
   )
   (symbol (lib_id "V2_Mechanical:Fiducial_Paste") (at 270.51 152.4 0) (unit 1)
-    (in_bom yes) (on_board yes) (dnp no)
+    (in_bom no) (on_board yes) (dnp no)
     (property "Reference" "FID101" (at 267.97 146.05 0)
       (effects (font (size 1.27 1.27)) (justify left))
@@
     )
     (property "Datasheet" "" (at 270.51 152.4 0)
+      (effects (font (size 1.27 1.27)) hide)
+    )
+    (property "Sim.Enable" "0" (at 270.51 152.4 0)
       (effects (font (size 1.27 1.27)) hide)
     )
@@
   )
   (symbol (lib_id "V2_Mechanical:Fiducial_Paste") (at 270.51 165.1 0) (unit 1)
-    (in_bom yes) (on_board yes) (dnp no)
+    (in_bom no) (on_board yes) (dnp no)
     (property "Reference" "FID102" (at 267.97 158.75 0)
       (effects (font (size 1.27 1.27)) (justify left))
@@
     )
     (property "Datasheet" "" (at 270.51 165.1 0)
+      (effects (font (size 1.27 1.27)) hide)
+    )
+    (property "Sim.Enable" "0" (at 270.51 165.1 0)
       (effects (font (size 1.27 1.27)) hide)
     )
@@
       (effects (font (size 1.27 1.27)) hide)
     )
+    (property "Sim.Enable" "0" (at 171.45 173.99 0)
+      (effects (font (size 1.27 1.27)) hide)
+    )
     (instances
       (project "strip"
@@
     )
     (property "Datasheet" "https://www.usb.org/sites/default/files/documents/usb_type-c.zip" (at 189.23 104.14 0)
+      (effects (font (size 1.27 1.27)) hide)
+    )
+    (property "Sim.Enable" "0" (at 185.42 104.14 0)
       (effects (font (size 1.27 1.27)) hide)
     )
@@
   )
   (symbol (lib_id "V2_Mechanical:Fiducial_Paste") (at 270.51 176.53 0) (unit 1)
-    (in_bom yes) (on_board yes) (dnp no)
+    (in_bom no) (on_board yes) (dnp no)
     (property "Reference" "FID103" (at 267.97 170.18 0)
       (effects (font (size 1.27 1.27)) (justify left))
@@
     )
     (property "Datasheet" "" (at 270.51 176.53 0)
+      (effects (font (size 1.27 1.27)) hide)
+    )
+    (property "Sim.Enable" "0" (at 270.51 176.53 0)
       (effects (font (size 1.27 1.27)) hide)
     )
@@
       (effects (font (size 1.27 1.27)) hide)
     )
+    (property "Sim.Enable" "0" (at 227.33 162.56 0)
+      (effects (font (size 1.27 1.27)) hide)
+    )
     (instances
       (project "strip"
@@
       (effects (font (size 1.27 1.27)) hide)
     )
+    (property "Sim.Enable" "0" (at 172.72 154.94 0)
+      (effects (font (size 1.27 1.27)) hide)
+    )
     (instances
       (project "strip"
@@
   (sheet (at 78.74 165.1) (size 22.86 7.62) (fields_autoplaced)
     (stroke (width 0.1524) (type solid))
-    (fill (color 0 0 0 0.0000))
+    (fill (color 255 255 194 1.0000))
     (property "Sheetname" "LED Strip" (at 78.74 164.3884 0)
       (effects (font (size 1.27 1.27)) (justify left bottom))
