File: strip-cover/strip-cover.kicad_pcb (KiCad board)
At the start: 2 copper layers, 66 x 18 mm, 7 parts

Commit message: Update to KiCad 7.0
Parts:
- H1: value MountingHole -> MountingHole_1mm; footprint V2_Mechanical:Mounting_Hole_1 -> V2_Mechanical:MountingHole_1mm
- H2, H3: value MountingHole_Pad -> MountingHole_2mm_Pad_5.2mm; footprint V2_Mechanical:Mounting_Hole_Pad_2-5.2 -> V2_Mechanical:Mounting_Hole_2mm_Pad_5.2mm
Connections:
- net /SHIELD renamed GND

Commit message: Refresh
Parts:
- H2, H3: value MountingHole_2mm_Pad_5.2mm -> Mounting_Hole; footprint V2_Mechanical:Mounting_Hole_2mm_Pad_5.2mm -> V2_Mechanical:MountingHole_2mm_Pad_5.2mm
Changed lines of the file:
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@@
   (setup
     (stackup
-      (layer "F.SilkS" (type "Top Silk Screen") (color "White") (color "White"))
+      (layer "F.SilkS" (type "Top Silk Screen") (color "White"))
       (layer "F.Paste" (type "Top Solder Paste"))
-      (layer "F.Mask" (type "Top Solder Mask") (color "Black") (color "Black") (thickness 0.01))
+      (layer "F.Mask" (type "Top Solder Mask") (color "Black") (thickness 0.01))
       (layer "F.Cu" (type "copper") (thickness 0.035))
       (layer "dielectric 1" (type "core") (thickness 1.5) (material "FR4") (epsilon_r 4.5) (loss_tangent 0.02))
       (layer "B.Cu" (type "copper") (thickness 0.035))
-      (layer "B.Mask" (type "Bottom Solder Mask") (color "Black") (color "Black") (thickness 0.01))
+      (layer "B.Mask" (type "Bottom Solder Mask") (color "Black") (thickness 0.01))
       (layer "B.Paste" (type "Bottom Solder Paste"))
-      (layer "B.SilkS" (type "Bottom Silk Screen") (color "White") (color "White"))
+      (layer "B.SilkS" (type "Bottom Silk Screen") (color "White"))
       (copper_finish "HAL lead-free")
       (dielectric_constraints no)
@@
     )
   )
-  (property "Order-Number" "ORDER-NUMBER")
+  (property "Order-Number" "JLCJLCJLCJLC")
   (net 0 "")
   (net 1 "GND")
@@
     (property "Sheetfile" "strip-cover.kicad_sch")
     (property "Sheetname" "")
+    (property "Sim.Enable" "0")
     (property "exclude_from_bom" "")
     (attr exclude_from_pos_files exclude_from_bom allow_missing_courtyard)
@@
       )
     )
-    (group "" (id 71708b3e-375b-440b-bea9-93cd9a6e1c5b)
+    (group "" (id 1b3a7dbc-baa6-4808-ad48-806962eb9f66)
       (members
-        120dcb07-45e9-4d19-aec7-f23f48531688
-        14b8ae9b-b15f-402f-b36d-3d93c7f64b3d
-        30b1d06c-3682-4567-b22c-a385330b6139
-        4513fe2b-bde4-48f6-83cf-dc29abe87574
-        59e5e18f-c197-4d61-9788-30023e77f1f4
-        6128f684-bb29-4847-bfaa-fc958a73dbfa
-        9d417248-38c6-4773-966f-f56951457e57
-        a8c176b9-a698-4a4d-9fe4-72a9d34c4cb7
-        f7d7be53-5bc0-4e99-8aee-9d7fb97aec04
-      )
-    )
-    (group "" (id a1293eb8-4120-4079-89c5-56358a96bb4b)
+        1cd7cf1f-6426-4427-bb97-afce74580622
+        273843fe-34c6-415d-8423-e38486aea3e5
+        48d20d61-02d2-4dad-8b53-aef08ba613f6
+        c7d50fcf-40ee-478c-92f1-9099cc6f0a59
+        db60cea2-c548-4a57-9ba1-c23fe130f3d9
+        defa8371-b27b-4109-aa27-4e08d9222f67
+        ee457ff1-c389-41a0-93e0-296a6f51f126
+        f81f2f80-5a48-473d-b987-a20a889eecd2
+        f9608ae1-68af-4185-bab5-d3bd900b93ea
+      )
+    )
+    (group "" (id 0eb86f08-f63c-4d3f-a69c-5cc530e4d1c4)
       (members
-        3677cccc-c48c-4e7a-852c-48295541531c
-        591f4be4-9f9a-4cc2-9a1b-1172305da87b
-        7b7b791c-8f26-4e2c-a847-a2cbb068d3c1
-        80af7dbf-53c2-4039-b38c-32fd42fee944
-        aa4ef438-3877-4747-8e46-5a1ec0321f29
-        aefd9f26-8222-499e-bba0-a869ac7ad742
-        caaf4ba8-a813-44e3-b97f-70f3145cdfe5
-        f5d58be6-27ea-4d1d-ac03-d61c1ff4db19
-        ff575b0a-7b4a-42b5-b947-e7503925c3d0
+        0a2ff4a4-4a40-4cd5-8877-06bae35613c5
+        395bccd8-3ccc-4c04-af4b-c0519924c150
+        4f47fd17-5d20-4e3e-9628-466c43585f04
+        59c31770-761e-4130-8131-b8485c3d81de
+        7b3e6d13-6676-4eec-9617-cf8dda2e6ac1
+        b5533a38-31d7-46af-a972-914ee6ad7d5b
+        d4c0d5be-9a46-4742-9d19-96c063e70d38
+        d5f675a7-5f48-4a22-ab82-b57c901e99dd
+        e15697a7-5b80-44b8-8d26-7201a7ab2ec3
       )
     )
@@
     (property "Sheetfile" "strip-cover.kicad_sch")
     (property "Sheetname" "")
+    (property "Sim.Enable" "0")
     (property "exclude_from_bom" "")
     (attr exclude_from_pos_files exclude_from_bom allow_missing_courtyard)
@@
     )
   )
-  (footprint "V2_Mechanical:Mounting_Hole_2mm_Pad_5.2mm" (layer "F.Cu")
+  (footprint "V2_Mechanical:MountingHole_2mm_Pad_5.2mm" (layer "F.Cu")
     (at 169 106)
     (property "Sheetfile" "strip-cover.kicad_sch")
     (property "Sheetname" "")
+    (property "Sim.Enable" "0")
+    (property "exclude_from_bom" "")
     (property "ki_description" "Mounting Hole with connection")
     (property "ki_keywords" "mounting hole")
+    (attr exclude_from_pos_files exclude_from_bom)
     (fp_text reference "H2" (at 0 -4 unlocked) (layer "F.SilkS") hide
         (effects (font (size 1 1) (thickness 0.15)))
     )
-    (fp_text value "MountingHole_2mm_Pad_5.2mm" (at 0 6 unlocked) (layer "F.Fab") hide
+    (fp_text value "Mounting_Hole" (at 0 6 unlocked) (layer "F.Fab") hide
         (effects (font (size 1 1) (thickness 0.15)))
     )
@@
     (fp_circle (center 0 0) (end 2.54 1.27)
       (stroke (width 0.05) (type solid)) (fill none) (layer "F.CrtYd"))
-    (pad "1" thru_hole custom (at 0 0) (size 5.4 5.4) (drill 2) (layers "*.Cu" "*.Mask") (remove_unused_layers) (keep_end_layers) (zone_layer_connections "F.Cu")
+    (pad "1" thru_hole custom (at 0 0) (size 5.4 5.4) (drill 2) (layers "*.Cu" "*.Mask") (remove_unused_layers) (keep_end_layers) (zone_layer_connections)
       (net 1 "GND") (pinfunction "1") (pintype "input") (zone_connect 2) (thermal_bridge_angle 45)
       (options (clearance outline) (anchor circle))
@@
     (property "Sheetfile" "strip-cover.kicad_sch")
     (property "Sheetname" "")
+    (property "Sim.Enable" "0")
+    (property "exclude_from_bom" "")
     (property "ki_description" "Mounting Hole without connection")
     (property "ki_keywords" "mounting hole")
+    (attr exclude_from_pos_files exclude_from_bom)
     (fp_text reference "H1" (at 0 -2 unlocked) (layer "F.SilkS") hide
         (effects (font (size 1 1) (thickness 0.15)))
@@
         (effects (font (size 1 1) (thickness 0.15)))
     )
-    (pad "" np_thru_hole circle (at 0 0) (size 1.2 1.2) (drill 1) (layers "*.Mask"))
+    (fp_circle (center 0 0) (end 0.6 0)
+      (stroke (width 0.05) (type default)) (fill none) (layer "F.CrtYd"))
+    (pad "" np_thru_hole circle (at 0 0) (size 1 1) (drill 1) (layers "*.Mask"))
   )
   (footprint "V2_PCB_Devices:PCB_Button-top" (layer "F.Cu")
@@
     (property "Sheetfile" "strip-cover.kicad_sch")
     (property "Sheetname" "")
+    (property "Sim.Enable" "0")
     (property "exclude_from_bom" "")
     (attr exclude_from_pos_files exclude_from_bom allow_missing_courtyard)
@@
     (fp_line (start 1.65 5.1) (end -1.65 5.1)
       (stroke (width 0.05) (type solid)) (layer "Edge.Cuts"))
-    (pad "" np_thru_hole circle (at -1.4 -4.85 90) (size 0.7 0.7) (drill 0.7) (layers "*.Cu" "*.Mask"))
-    (pad "" np_thru_hole circle (at -1.4 4.85 90) (size 0.7 0.7) (drill 0.7) (layers "*.Cu" "*.Mask"))
-    (pad "" np_thru_hole circle (at 1.4 -4.85 90) (size 0.7 0.7) (drill 0.7) (layers "*.Cu" "*.Mask"))
-    (pad "" np_thru_hole circle (at 1.4 4.85 90) (size 0.7 0.7) (drill 0.7) (layers "*.Cu" "*.Mask"))
+    (pad "" np_thru_hole circle (at -1.4 -4.85 90) (size 0.7 0.7) (drill 0.7) (layers "*.Mask"))
+    (pad "" np_thru_hole circle (at -1.4 4.85 90) (size 0.7 0.7) (drill 0.7) (layers "*.Mask"))
+    (pad "" np_thru_hole circle (at 1.4 -4.85 90) (size 0.7 0.7) (drill 0.7) (layers "*.Mask"))
+    (pad "" np_thru_hole circle (at 1.4 4.85 90) (size 0.7 0.7) (drill 0.7) (layers "*.Mask"))
   )
-  (footprint "V2_Mechanical:Mounting_Hole_2mm_Pad_5.2mm" (layer "F.Cu")
+  (footprint "V2_Mechanical:MountingHole_2mm_Pad_5.2mm" (layer "F.Cu")
     (at 131 106)
     (property "Sheetfile" "strip-cover.kicad_sch")
     (property "Sheetname" "")
+    (property "Sim.Enable" "0")
+    (property "exclude_from_bom" "")
     (property "ki_description" "Mounting Hole with connection")
     (property "ki_keywords" "mounting hole")
+    (attr exclude_from_pos_files exclude_from_bom)
     (fp_text reference "H3" (at 0 -4 unlocked) (layer "F.SilkS") hide
         (effects (font (size 1 1) (thickness 0.15)))
     )
-    (fp_text value "MountingHole_2mm_Pad_5.2mm" (at 0 6 unlocked) (layer "F.Fab") hide
+    (fp_text value "Mounting_Hole" (at 0 6 unlocked) (layer "F.Fab") hide
         (effects (font (size 1 1) (thickness 0.15)))
     )
@@
     (fp_circle (center 0 0) (end 2.54 1.27)
       (stroke (width 0.05) (type solid)) (fill none) (layer "F.CrtYd"))
-    (pad "1" thru_hole custom (at 0 0) (size 5.4 5.4) (drill 2) (layers "*.Cu" "*.Mask") (remove_unused_layers) (keep_end_layers) (zone_layer_connections "F.Cu")
+    (pad "1" thru_hole custom (at 0 0) (size 5.4 5.4) (drill 2) (layers "*.Cu" "*.Mask") (remove_unused_layers) (keep_end_layers) (zone_layer_connections)
       (net 1 "GND") (pinfunction "1") (pintype "input") (zone_connect 2) (thermal_bridge_angle 45)
       (options (clearance outline) (anchor circle))
@@
     (property "Sheetfile" "strip-cover.kicad_sch")
     (property "Sheetname" "")
+    (property "Sim.Enable" "0")
     (property "exclude_from_bom" "")
-    (attr exclude_from_pos_files exclude_from_bom allow_missing_courtyard)
+    (attr exclude_from_pos_files exclude_from_bom)
     (fp_text reference "INFO1" (at 0 1.77 unlocked) (layer "B.SilkS") hide
         (effects (font (size 1 1) (thickness 0.15)) (justify mirror))
@@
         (effects (font (size 0.8 0.8) (thickness 0.12)) (justify mirror))
     )
+    (fp_rect (start -7 0.75) (end 7 -0.75)
+      (stroke (width 0.05) (type default)) (fill none) (layer "B.CrtYd"))
   )
   (gr_line (start 117 98) (end 117 114)
